Commit message: added description

File: site_configs/tormach_za6_base_config/description/za6.xacro (robot description, xacro)
@@ -135,5 +135,5 @@
   </link>
   <joint name="table_joint" type="fixed">
-    <parent link="base_link" />
+    <parent link="world" />
     <child link="environment" />
     <origin rpy="0 0 0" xyz="0 0 -0.05" />
