Commit message: Add `manual_grasp_link` to kinematic chain  FIXME
Add `manual_grasp_link` to description and update MoveIt config.  This
is broken.

File: za6_description/urdf/za6_macro.xacro (robot description, xacro)
@@ -242,4 +242,11 @@
       </joint>
     </xacro:unless>
+    <!-- MoveIt Studio 'manual_grasp_link' for planning -->
+    <link name="manual_grasp_link"/>
+    <joint name="${prefix}manual_grasp_link-tool0" type="fixed">
+      <origin xyz="0 0 0" rpy="0 0 0" />
+      <parent link="${prefix}tool0" />
+      <child link="${prefix}manual_grasp_link" />
+    </joint>
   </xacro:macro>
 </robot>

Commit message: Added waypoints and updated objectives

File: za6_description/urdf/za6_macro.xacro (robot description, xacro)
@@ -243,5 +243,5 @@
     </xacro:unless>
     <!-- MoveIt Studio 'manual_grasp_link' for planning -->
-    <link name="manual_grasp_link"/>
+    <link name="manual_grasp_link" />
     <joint name="${prefix}manual_grasp_link-tool0" type="fixed">
       <origin xyz="0 0 0" rpy="0 0 0" />
