Commit message: za6_description:  Move URDF `manual_grasp_link` out of ZA6 xacro
Following the Studio example, put the `manual_grasp_link` in the
top-level `xacro` file.

File: za6_description/urdf/za6.xacro (robot description, xacro)
@@ -101,3 +101,10 @@
     <child link="$(arg prefix)base_link"/>
   </joint>
+  <!-- MoveIt Studio 'manual_grasp_link' for planning -->
+  <link name="manual_grasp_link" />
+  <joint name="$(arg prefix)manual_grasp_link-tool0" type="fixed">
+    <origin xyz="0 0 0" rpy="0 0 0" />
+    <parent link="$(arg prefix)tool0" />
+    <child link="$(arg prefix)manual_grasp_link" />
+  </joint>
 </robot>

File: za6_description/urdf/za6_macro.xacro (robot description, xacro)
@@ -242,11 +242,4 @@
       </joint>
     </xacro:unless>
-    <!-- MoveIt Studio 'manual_grasp_link' for planning -->
-    <link name="manual_grasp_link" />
-    <joint name="${prefix}manual_grasp_link-tool0" type="fixed">
-      <origin xyz="0 0 0" rpy="0 0 0" />
-      <parent link="${prefix}tool0" />
-      <child link="${prefix}manual_grasp_link" />
-    </joint>
   </xacro:macro>
 </robot>

Commit message: za6_description:  Add za6_tools grippers into URDFs

File: za6_description/urdf/za6.xacro (robot description, xacro)
@@ -35,4 +35,10 @@
   <xacro:arg name="limit_joint_6_velocity" default="6.2"/>
   <xacro:arg name="limit_joint_6_effort" default="1000.0"/>
+  <xacro:arg name="gripper" default="none"/>
+  <xacro:property name="gripper" value="$(arg gripper)"/>
+  <!-- MoveIt Studio web preview gripper model -->
+  <xacro:attribute
+      name="web_ui_gripper"
+      value="$(find za6_tools)/urdf/${gripper}.urdf"/>
   <xacro:include filename="$(find za6_description)/urdf/za6_macro.xacro"/>
   <xacro:za6
@@ -41,4 +47,5 @@
       tool0_rot="0 0 0"
       tool0_fixed="$(arg fixed_tool)"
+      gripper="${gripper}"
       limit_joint_1_lower="$(arg limit_joint_1_lower)"
       limit_joint_1_upper="$(arg limit_joint_1_upper)"
@@ -108,5 +115,5 @@
   <joint name="$(arg prefix)manual_grasp_joint" type="fixed">
     <origin xyz="0 0 0" rpy="0 0 0" />
-    <parent link="$(arg prefix)tool0" />
+    <parent link="$(arg prefix)grasp_link" />
     <child link="$(arg prefix)manual_grasp_link" />
   </joint>

File: za6_description/urdf/za6_macro.xacro (robot description, xacro)
@@ -2,6 +2,9 @@
 <robot xmlns:xacro="http://www.ros.org/wiki/xacro">
   <xacro:macro name="za6" params="
-    prefix tool0_trans tool0_rot
+    prefix
+    tool0_trans
+    tool0_rot
     tool0_fixed:=True
+    gripper:=''
     limit_joint_1_lower:=-2.96
     limit_joint_1_upper:=2.96
@@ -243,4 +246,21 @@
       </joint>
     </xacro:unless>
+    <xacro:unless value="${gripper == '' or gripper == 'none'}">
+      <!-- Gripper params supplied in macro call -->
+      <xacro:include filename="$(find za6_tools)/urdf/${gripper}_macro.xacro"/>
+      <!-- Attach gripper to ZA6 "flange" link -->
+      <xacro:element xacro:name="xacro:${gripper}_macro"
+                     prefix="${prefix}"
+                     connected_to="${prefix}flange"/>
+    </xacro:unless>
+    <xacro:if value="${gripper == '' or gripper == 'none'}">
+      <!-- No gripper params; create grasp_link & connect to flange -->
+      <link name="grasp_link" />
+      <joint name="${prefix}grasp_joint" type="fixed">
+        <origin xyz="0 0 0" rpy="0 0 0" />
+        <parent link="${prefix}flange" />
+        <child link="${prefix}grasp_link" />
+      </joint>
+    </xacro:if>
   </xacro:macro>
 </robot>

Commit message: za6_description:  FIXME tweak URDF

File: za6_description/urdf/za6.xacro (robot description, xacro)
@@ -36,9 +36,8 @@
   <xacro:arg name="limit_joint_6_effort" default="1000.0"/>
   <xacro:arg name="gripper" default="none"/>
-  <xacro:property name="gripper" value="$(arg gripper)"/>
   <!-- MoveIt Studio web preview gripper model -->
   <xacro:attribute
       name="web_ui_gripper"
-      value="$(find za6_tools)/urdf/${gripper}.urdf"/>
+      value="package://za6_tools/urdf/$(arg gripper).urdf"/>
   <xacro:include filename="$(find za6_description)/urdf/za6_macro.xacro"/>
   <xacro:za6
@@ -47,5 +46,5 @@
       tool0_rot="0 0 0"
       tool0_fixed="$(arg fixed_tool)"
-      gripper="${gripper}"
+      gripper="$(arg gripper)"
       limit_joint_1_lower="$(arg limit_joint_1_lower)"
       limit_joint_1_upper="$(arg limit_joint_1_upper)"
@@ -115,5 +114,5 @@
   <joint name="$(arg prefix)manual_grasp_joint" type="fixed">
     <origin xyz="0 0 0" rpy="0 0 0" />
-    <parent link="$(arg prefix)grasp_link" />
+    <parent link="$(arg prefix)tool0" />
     <child link="$(arg prefix)manual_grasp_link" />
   </joint>

File: za6_description/urdf/za6_macro.xacro (robot description, xacro)
@@ -232,5 +232,5 @@
     <link name="${prefix}tool0" />
     <xacro:if value="${tool0_fixed}">
-      <joint name="${prefix}link_6_tool0" type="fixed">
+      <joint name="${prefix}flange_tool0" type="fixed">
         <!-- marker -->
         <origin xyz="${tool0_trans}" rpy="${tool0_rot}" />
@@ -240,5 +240,5 @@
     </xacro:if>
     <xacro:unless value="${tool0_fixed}">
-      <joint name="${prefix}link_6_tool0" type="floating">
+      <joint name="${prefix}flange_tool0" type="floating">
         <origin xyz="0 0 0" rpy="0 0 0" />
         <parent link="${prefix}flange" />
@@ -246,20 +246,20 @@
       </joint>
     </xacro:unless>
-    <xacro:unless value="${gripper == '' or gripper == 'none'}">
+    <xacro:unless value="${gripper == ''}">
       <!-- Gripper params supplied in macro call -->
       <xacro:include filename="$(find za6_tools)/urdf/${gripper}_macro.xacro"/>
-      <!-- Attach gripper to ZA6 "flange" link -->
+      <!-- Attach gripper to ZA6 "tool0" link -->
       <xacro:element xacro:name="xacro:${gripper}_macro"
                      prefix="${prefix}"
-                     connected_to="${prefix}flange"/>
+                     connected_to="${prefix}tool0"/>
     </xacro:unless>
-    <xacro:if value="${gripper == '' or gripper == 'none'}">
-      <!-- No gripper params; create grasp_link & connect to flange -->
-      <link name="grasp_link" />
-      <joint name="${prefix}grasp_joint" type="fixed">
-        <origin xyz="0 0 0" rpy="0 0 0" />
-        <parent link="${prefix}flange" />
-        <child link="${prefix}grasp_link" />
-      </joint>
+    <xacro:if value="${gripper == ''}">
+      <!-- No gripper params; use 'none' gripper URDF -->
+      <!-- Gripper params supplied in macro call -->
+      <xacro:include filename="$(find za6_tools)/urdf/none_macro.xacro"/>
+      <!-- Attach gripper to ZA6 "tool0" link -->
+      <xacro:element xacro:name="xacro:none_macro"
+                     prefix="${prefix}"
+                     connected_to="${prefix}tool0"/>
     </xacro:if>
   </xacro:macro>

Commit message: za6_description:  Fix tool grasp position FIXME
Fix MoveIt Studio iMarker to center on gripper grasp link rather than
on flange.

File: za6_description/urdf/za6.xacro (robot description, xacro)
@@ -114,5 +114,5 @@
   <joint name="$(arg prefix)manual_grasp_joint" type="fixed">
     <origin xyz="0 0 0" rpy="0 0 0" />
-    <parent link="$(arg prefix)tool0" />
+    <parent link="$(arg prefix)grasp_link" />
     <child link="$(arg prefix)manual_grasp_link" />
   </joint>

Commit message: za_description:  Tweak URDFs
Use `za_tools` CMake function for looping over gripper models in
tests.

Remove MoveIt Studio specific config; that will move to Studio-related
packages.

File: za6_description/urdf/za6.xacro (robot description, xacro)
@@ -36,8 +36,4 @@
   <xacro:arg name="limit_joint_6_effort" default="1000.0"/>
   <xacro:arg name="gripper" default="none"/>
-  <!-- MoveIt Studio web preview gripper model -->
-  <xacro:attribute
-      name="web_ui_gripper"
-      value="package://za6_tools/urdf/$(arg gripper).urdf"/>
   <xacro:include filename="$(find za6_description)/urdf/za6_macro.xacro"/>
   <xacro:za6
@@ -109,11 +105,3 @@
     <child link="$(arg prefix)base_link"/>
   </joint>
-  <!-- Moveit Studio requires a link name called manual_grasp_link to
-       perform quick tasks such as inspect surface -->
-  <link name="manual_grasp_link" />
-  <joint name="$(arg prefix)manual_grasp_joint" type="fixed">
-    <origin xyz="0 0 0" rpy="0 0 0" />
-    <parent link="$(arg prefix)grasp_link" />
-    <child link="$(arg prefix)manual_grasp_link" />
-  </joint>
 </robot>
