Commit message: Add updated SRDFs for all tools in Studio config; clean up tools

File: za6_tools/urdf/pivot_gripper.xacro (robot description, xacro)
@@ -3,13 +3,8 @@
   <xacro:arg name="prefix" default=""/>
   <xacro:include filename="$(find za6_tools)/urdf/pivot_gripper_macro.xacro"/>
+  <!-- 'flange' frame: default pose reference frame -->
+  <link name="flange" />
   <xacro:pivot_gripper_macro
       prefix="$(arg prefix)"
       connected_to="flange-$(arg prefix)za6_pivot_adapter"/>
-  <!-- 'flange' frame: default pose reference frame -->
-  <link name="flange" />
-  <joint name="flange-$(arg prefix)za6_pivot_adapter" type="fixed">
-    <origin xyz="0 0 0" rpy="0 0 ${pi}"/>
-    <axis xyz="0 0 1"/>
-    <parent link="flange"/>
-  </joint>
 </robot>

File: za6_tools/urdf/pivot_gripper_macro.xacro (robot description, xacro)
@@ -3,5 +3,5 @@
   <xacro:macro name="pivot_gripper_macro" params="prefix connected_to">
     <material name="${prefix}Aluminium">
-      <color rgba="0.9 0.9 0.9 0.99"/>
+      <color rgba="0.9 0.9 0.9 1.0"/>
     </material>
     <!-- link list -->
@@ -87,12 +87,12 @@
     </link>
     <!-- joint list -->
-    <joint name="${prefix}adapter-pivot_gripper_base" type="fixed">
+    <joint name="${prefix}pivot_gripper_base_joint" type="fixed">
       <parent link="${connected_to}"/>
       <child link="${prefix}pivot_gripper_base"/>
-      <axis xyz="0 0 0"/>
+      <axis xyz="0 0 1"/>
       <origin rpy="0.0 0.0 0.0" xyz="0 0 0"/>
     </joint>
     <joint
-        name="${prefix}pivot_gripper_base-pivot_gripper_finger_left1"
+        name="${prefix}pivot_gripper_finger_left1_joint"
         type="fixed">
       <parent link="${prefix}pivot_gripper_base" />
@@ -102,5 +102,5 @@
     </joint>
     <joint
-        name="${prefix}pivot_gripper_base-pivot_gripper_finger_right1"
+        name="${prefix}pivot_gripper_finger_right1_joint"
         type="fixed">
       <parent link="${prefix}pivot_gripper_base" />
@@ -110,5 +110,5 @@
     </joint>
     <joint
-        name="${prefix}pivot_gripper_base-pivot_gripper_finger_left2"
+        name="${prefix}pivot_gripper_finger_left2_joint"
         type="fixed">
       <parent link="${prefix}pivot_gripper_base" />
@@ -118,5 +118,5 @@
     </joint>
     <joint
-        name="${prefix}pivot_gripper_base-pivot_gripper_finger_right2"
+        name="${prefix}pivot_gripper_finger_right2_joint"
         type="fixed">
       <parent link="${prefix}pivot_gripper_base" />

File: za6_tools/urdf/pivot_gripper_standalone.xacro (robot description, xacro)
@@ -2,7 +2,4 @@
 <robot name="za6" xmlns:xacro="http://ros.org/wiki/xacro">
   <xacro:include filename="$(find za6_tools)/urdf/pivot_gripper_macro.xacro"/>
-  <xacro:pivot_gripper_macro
-      prefix=""
-      connected_to="base_link"/>
   <material name="main_Red">
     <color rgba="0.7 0.0 0.0 0.99"/>
@@ -22,3 +19,6 @@
     <child link="base_link"/>
   </joint>
+  <xacro:pivot_gripper_macro
+      prefix=""
+      connected_to="base_link"/>
 </robot>

File: za6_tools/urdf/robotiq_hand_e.xacro (robot description, xacro)
@@ -3,12 +3,8 @@
   <xacro:arg name="prefix" default=""/>
   <xacro:include filename="$(find za6_tools)/urdf/robotiq_hand_e_macro.xacro"/>
-  <xacro:robotiq_hand_e_macro prefix="$(arg prefix)"/>
   <!-- 'flange' frame: default pose reference frame -->
   <link name="flange" />
-  <joint name="flange-$(arg prefix)hand_e_body" type="fixed">
-    <origin xyz="0 0 0" rpy="0 0 ${-pi/2.0}"/>
-    <axis xyz="0 0 1"/>
-    <parent link="flange"/>
-    <child link="$(arg prefix)hand_e_body"/>
-  </joint>
+  <xacro:robotiq_hand_e_macro
+      prefix="$(arg prefix)"
+      connected_to="$(arg prefix)flange"/>
 </robot>

File: za6_tools/urdf/robotiq_hand_e_macro.xacro (robot description, xacro)
@@ -1,5 +1,5 @@
 <?xml version="1.0"?>
 <robot xmlns:xacro="http://www.ros.org/wiki/xacro">
-  <xacro:macro name="robotiq_hand_e_macro" params="prefix">
+  <xacro:macro name="robotiq_hand_e_macro" params="prefix connected_to">
     <material name="${prefix}Aluminium">
       <color rgba="0.9 0.9 0.9 0.99"/>
@@ -60,4 +60,10 @@
     </link>
     <!-- joint list -->
+    <joint name="${prefix}flange-hand_e_body" type="fixed">
+      <parent link="${connected_to}"/>
+      <child link="${prefix}hand_e_body"/>
+      <axis xyz="0 0 1"/>
+      <origin rpy="0 0 ${-pi/2.0}" xyz="0 0 0"/>
+    </joint>
     <joint name="${prefix}hand_e_body-hand_e_finger_left" type="fixed">
       <parent link="${prefix}hand_e_body" />

File: za6_tools/urdf/robotiq_hand_e_standalone.xacro (robot description, xacro)
@@ -2,5 +2,4 @@
 <robot name="za6" xmlns:xacro="http://ros.org/wiki/xacro">
   <xacro:include filename="$(find za6_tools)/urdf/robotiq_hand_e_macro.xacro"/>
-  <xacro:robotiq_hand_e_macro prefix=""/>
   <material name="main_Red">
     <color rgba="0.7 0.0 0.0 0.99"/>
@@ -20,8 +19,6 @@
     <child link="base_link"/>
   </joint>
-  <joint name="base-adapter" type="fixed">
-    <parent link="base_link"/>
-    <child link="za6_robotiq_adapter"/>
-    <origin rpy="0 0 0" xyz="0 0 0.1"/>
-  </joint>
+  <xacro:robotiq_hand_e_macro
+      prefix=""
+      connected_to="base_link"/>
 </robot>

File: za6_tools/urdf/versabuilt_multigrip.xacro (robot description, xacro)
@@ -2,13 +2,10 @@
 <robot name="za6" xmlns:xacro="http://ros.org/wiki/xacro">
   <xacro:arg name="prefix" default=""/>
-  <xacro:include filename="$(find za6_tools)/urdf/versabuilt_multigrip_macro.xacro"/>
-  <xacro:versabuilt_multigrip_macro prefix="$(arg prefix)"/>
+  <xacro:include
+      filename="$(find za6_tools)/urdf/versabuilt_multigrip_macro.xacro"/>
   <!-- 'flange' frame: default pose reference frame -->
   <link name="flange" />
-  <joint name="flange-$(arg prefix)za6_multigrip_adapter" type="fixed">
-    <origin xyz="0 0 0" rpy="0 0 ${pi}"/>
-    <axis xyz="0 0 1"/>
-    <parent link="flange"/>
-    <child link="$(arg prefix)za6_multigrip_adapter"/>
-  </joint>
+  <xacro:versabuilt_multigrip_macro
+      prefix="$(arg prefix)"
+      connected_to="flange"/>
 </robot>

File: za6_tools/urdf/versabuilt_multigrip_macro.xacro (robot description, xacro)
@@ -1,5 +1,5 @@
 <?xml version="1.0"?>
 <robot xmlns:xacro="http://www.ros.org/wiki/xacro">
-  <xacro:macro name="versabuilt_multigrip_macro" params="prefix">
+  <xacro:macro name="versabuilt_multigrip_macro" params="prefix connected_to">
     <material name="${prefix}Aluminium">
       <color rgba="0.9 0.9 0.9 0.99"/>
@@ -49,4 +49,10 @@
     </link>
     <!-- joint list -->
+    <joint name="${prefix}flange-multigrip_adapter" type="fixed">
+      <parent link="${connected_to}"/>
+      <child link="${prefix}za6_multigrip_adapter"/>
+      <axis xyz="0 0 0"/>
+      <origin rpy="0.0 0.0 0.0" xyz="0 0 0"/>
+    </joint>
     <joint name="${prefix}adapter-multigrip_base_and_fixed_jaw" type="fixed">
       <parent link="${prefix}za6_multigrip_adapter"/>
@@ -55,9 +61,9 @@
       <origin xyz="0 0 0" rpy="${pi/2.0} -${pi/2.0} -${pi/2.0}"/>
     </joint>
-    <joint name="${prefix}multigrip_base_and_fixed_jaw-multigrip_moving_jaw" type="fixed">
+    <joint name="${prefix}multigrip_moving_jaw_joint" type="fixed">
       <parent link="${prefix}multigrip_base_and_fixed_jaw" />
       <child link="${prefix}multigrip_moving_jaw" />
       <axis xyz="0 0 1"/>
-      <origin xyz="0.0 0 0.0" rpy="0 0 0" />
+      <origin xyz="0.0 0 0.0" rpy="0 0 ${pi}" />
     </joint>
   </xacro:macro>

File: za6_tools/urdf/versabuilt_multigrip_standalone.xacro (robot description, xacro)
@@ -1,6 +1,6 @@
 <?xml version="1.0" ?>
 <robot name="za6" xmlns:xacro="http://ros.org/wiki/xacro">
-  <xacro:include filename="$(find za6_tools)/urdf/versabuilt_multigrip_macro.xacro"/>
-  <xacro:versabuilt_multigrip_macro prefix=""/>
+  <xacro:include
+      filename="$(find za6_tools)/urdf/versabuilt_multigrip_macro.xacro"/>
   <material name="main_Red">
     <color rgba="0.7 0.0 0.0 0.99"/>
@@ -20,8 +20,6 @@
     <child link="base_link"/>
   </joint>
-  <joint name="base-adapter" type="fixed">
-    <parent link="base_link"/>
-    <child link="za6_multigrip_adapter"/>
-    <origin rpy="0 0 0" xyz="0 0 0.1"/>
-  </joint>
+  <xacro:versabuilt_multigrip_macro
+      prefix=""
+      connected_to="base_link"/>
 </robot>
