Commit message: za6_tools:  Build static urdfs
For Studio, which can take a `<xacro:attribute name="web_ui_gripper"
value="some.urdf" />` arg for the web interface visual, which is a
Robotiq by default.

File: za6_tools/urdf/pivot_gripper.urdf.xacro (robot description, xacro)
@@ -2,9 +2,9 @@
 <robot name="za6" xmlns:xacro="http://www.ros.org/wiki/xacro">
   <xacro:arg name="prefix" default=""/>
-  <xacro:include filename="$(find za6_tools)/urdf/pivot_gripper_macro.xacro"/>
+  <xacro:include filename="$(cwd)/urdf/pivot_gripper_macro.xacro"/>
   <!-- 'flange' frame: default pose reference frame -->
   <link name="flange" />
   <xacro:pivot_gripper_macro
       prefix="$(arg prefix)"
-      connected_to="flange-$(arg prefix)za6_pivot_adapter"/>
+      connected_to="$(arg prefix)flange"/>
 </robot>

File: za6_tools/urdf/pivot_gripper_macro.xacro (robot description, xacro)
@@ -125,4 +125,11 @@
       <origin xyz="-0.0843 -0.0053 0.031" rpy="0 -${pi/2.0} 0" />
     </joint>
+    <!-- Attach grasp_link to gripper base for now -->
+    <link name="grasp_link" />
+    <joint name="grasp_joint" type="fixed">
+      <parent link="$(arg prefix)pivot_gripper_base" />
+      <child link="grasp_link" />
+      <origin xyz="0.0 0.0 0.0" rpy="0.0 0.0 0.0" />
+    </joint>
   </xacro:macro>
 </robot>

File: za6_tools/urdf/pivot_gripper_standalone.xacro (robot description, xacro)
@@ -3,5 +3,5 @@
   <xacro:include filename="$(find za6_tools)/urdf/pivot_gripper_macro.xacro"/>
   <material name="main_Red">
-    <color rgba="0.7 0.0 0.0 0.99"/>
+    <color rgba="0.7 0.0 0.0 1.0"/>
   </material>
   <link name="world"/>

File: za6_tools/urdf/robotiq_hand_e.urdf.xacro (robot description, xacro)
@@ -2,5 +2,5 @@
 <robot name="za6" xmlns:xacro="http://www.ros.org/wiki/xacro">
   <xacro:arg name="prefix" default=""/>
-  <xacro:include filename="$(find za6_tools)/urdf/robotiq_hand_e_macro.xacro"/>
+  <xacro:include filename="$(cwd)/urdf/robotiq_hand_e_macro.xacro"/>
   <!-- 'flange' frame: default pose reference frame -->
   <link name="flange" />

File: za6_tools/urdf/robotiq_hand_e_macro.xacro (robot description, xacro)
@@ -3,8 +3,8 @@
   <xacro:macro name="robotiq_hand_e_macro" params="prefix connected_to">
     <material name="${prefix}Aluminium">
-      <color rgba="0.9 0.9 0.9 0.99"/>
+      <color rgba="0.9 0.9 0.9 1.0"/>
     </material>
     <material name="${prefix}Black">
-      <color rgba="0.1 0.1 0.1 0.99"/>
+      <color rgba="0.1 0.1 0.1 1.0"/>
     </material>
     <!-- link list -->
@@ -78,4 +78,11 @@
       <origin xyz="-0.025 0 0.0965" rpy="0 0 -${pi/2.0}" />
     </joint>
+    <!-- Attach grasp_link to gripper body for now -->
+    <link name="grasp_link" />
+    <joint name="grasp_joint" type="fixed">
+      <parent link="${prefix}hand_e_body" />
+      <child link="grasp_link" />
+      <origin xyz="0.0 0.0 0.0" rpy="0.0 0.0 0.0" />
+    </joint>
   </xacro:macro>
 </robot>

File: za6_tools/urdf/robotiq_hand_e_standalone.xacro (robot description, xacro)
@@ -3,5 +3,5 @@
   <xacro:include filename="$(find za6_tools)/urdf/robotiq_hand_e_macro.xacro"/>
   <material name="main_Red">
-    <color rgba="0.7 0.0 0.0 0.99"/>
+    <color rgba="0.7 0.0 0.0 1.0"/>
   </material>
   <link name="world"/>

File: za6_tools/urdf/versabuilt_multigrip.urdf.xacro (robot description, xacro)
@@ -3,9 +3,9 @@
   <xacro:arg name="prefix" default=""/>
   <xacro:include
-      filename="$(find za6_tools)/urdf/versabuilt_multigrip_macro.xacro"/>
+      filename="$(cwd)/urdf/versabuilt_multigrip_macro.xacro"/>
   <!-- 'flange' frame: default pose reference frame -->
   <link name="flange" />
   <xacro:versabuilt_multigrip_macro
       prefix="$(arg prefix)"
-      connected_to="flange"/>
+      connected_to="$(arg prefix)flange"/>
 </robot>

File: za6_tools/urdf/versabuilt_multigrip_macro.xacro (robot description, xacro)
@@ -3,5 +3,5 @@
   <xacro:macro name="versabuilt_multigrip_macro" params="prefix connected_to">
     <material name="${prefix}Aluminium">
-      <color rgba="0.9 0.9 0.9 0.99"/>
+      <color rgba="0.9 0.9 0.9 1.0"/>
     </material>
     <!-- link list -->
@@ -67,4 +67,11 @@
       <origin xyz="0.0 0 0.0" rpy="0 0 ${pi}" />
     </joint>
+    <!-- Attach grasp_link to multigrip base for now -->
+    <link name="grasp_link" />
+    <joint name="grasp_joint" type="fixed">
+      <parent link="$(arg prefix)multigrip_base_and_fixed_jaw" />
+      <child link="grasp_link" />
+      <origin xyz="0.0 0.0 0.0" rpy="0.0 0.0 0.0" />
+    </joint>
   </xacro:macro>
 </robot>

File: za6_tools/urdf/versabuilt_multigrip_standalone.xacro (robot description, xacro)
@@ -4,5 +4,5 @@
       filename="$(find za6_tools)/urdf/versabuilt_multigrip_macro.xacro"/>
   <material name="main_Red">
-    <color rgba="0.7 0.0 0.0 0.99"/>
+    <color rgba="0.7 0.0 0.0 1.0"/>
   </material>
   <link name="world"/>

Commit message: za6_tools:  Fix tool top-level xacro for build & display, both
When running the `display_*.launch` files, `$(cwd)` doesn't work,
because the current directory is the `urdf/` directory.  When building
the static URDF files from `CMakeLists.txt`, `$(find za_tools)`
doesn't work, because it refers to itself, which is currently being
built.

Fix both cases by hacking in a `_build` arg to select the appropriate
method.

File: za6_tools/urdf/pivot_gripper.urdf.xacro (robot description, xacro)
@@ -2,5 +2,17 @@
 <robot name="za6" xmlns:xacro="http://www.ros.org/wiki/xacro">
   <xacro:arg name="prefix" default=""/>
-  <xacro:include filename="$(cwd)/urdf/pivot_gripper_macro.xacro"/>
+  <xacro:arg name="_build" default="false"/>
+  <xacro:if value="$(arg _build)">
+    <xacro:include filename="$(cwd)/urdf/pivot_gripper_macro.xacro"/>
+  </xacro:if>
+  <xacro:unless value="$(arg _build)">
+    <xacro:include filename="$(find za6_tools)/urdf/pivot_gripper_macro.xacro"/>
+  </xacro:unless>
+  <link name="tool0"/>
+  <joint name="flange-tool0" type="fixed">
+    <parent link="manual_grasp_link"/>
+    <child link="tool0"/>
+    <origin rpy="0.08726646259971647 0 -3.141592653589793" xyz="0.0 -0.016124 -0.18430"/>
+  </joint>
   <!-- 'flange' frame: default pose reference frame -->
   <link name="flange" />
@@ -8,3 +20,11 @@
       prefix="$(arg prefix)"
       connected_to="$(arg prefix)flange"/>
+  <!-- Moveit Studio requires a link name called manual_grasp_link to
+       perform quick tasks such as inspect surface -->
+  <link name="manual_grasp_link" />
+  <joint name="$(arg prefix)manual_grasp_joint" type="fixed">
+    <origin xyz="0 0 0" rpy="0 0 0" />
+    <parent link="$(arg prefix)grasp_link" />
+    <child link="$(arg prefix)manual_grasp_link" />
+  </joint>
 </robot>

File: za6_tools/urdf/robotiq_hand_e.urdf.xacro (robot description, xacro)
@@ -2,5 +2,17 @@
 <robot name="za6" xmlns:xacro="http://www.ros.org/wiki/xacro">
   <xacro:arg name="prefix" default=""/>
-  <xacro:include filename="$(cwd)/urdf/robotiq_hand_e_macro.xacro"/>
+  <xacro:arg name="_build" default="false"/>
+  <xacro:if value="$(arg _build)">
+    <xacro:include filename="$(cwd)/urdf/robotiq_hand_e_macro.xacro"/>
+  </xacro:if>
+  <xacro:unless value="$(arg _build)">
+    <xacro:include filename="$(find za6_tools)/urdf/robotiq_hand_e_macro.xacro"/>
+  </xacro:unless>
+  <link name="tool0"/>
+  <joint name="flange-tool0" type="fixed">
+    <parent link="manual_grasp_link"/>
+    <child link="tool0"/>
+    <origin rpy="0.08726646259971647 0 -3.141592653589793" xyz="0.0 -0.016124 -0.18430"/>
+  </joint>
   <!-- 'flange' frame: default pose reference frame -->
   <link name="flange" />
@@ -8,3 +20,11 @@
       prefix="$(arg prefix)"
       connected_to="$(arg prefix)flange"/>
+  <!-- Moveit Studio requires a link name called manual_grasp_link to
+       perform quick tasks such as inspect surface -->
+  <link name="manual_grasp_link" />
+  <joint name="$(arg prefix)manual_grasp_joint" type="fixed">
+    <origin xyz="0 0 0" rpy="0 0 0" />
+    <parent link="$(arg prefix)grasp_link" />
+    <child link="$(arg prefix)manual_grasp_link" />
+  </joint>
 </robot>

File: za6_tools/urdf/versabuilt_multigrip.urdf.xacro (robot description, xacro)
@@ -2,6 +2,18 @@
 <robot name="za6" xmlns:xacro="http://ros.org/wiki/xacro">
   <xacro:arg name="prefix" default=""/>
-  <xacro:include
-      filename="$(cwd)/urdf/versabuilt_multigrip_macro.xacro"/>
+  <xacro:arg name="_build" default="false"/>
+  <xacro:if value="$(arg _build)">
+    <xacro:include filename="$(cwd)/urdf/versabuilt_multigrip_macro.xacro"/>
+  </xacro:if>
+  <xacro:unless value="$(arg _build)">
+    <xacro:include
+        filename="$(find za6_tools)/urdf/versabuilt_multigrip_macro.xacro"/>
+  </xacro:unless>
+  <link name="tool0"/>
+  <joint name="flange-tool0" type="fixed">
+    <parent link="manual_grasp_link"/>
+    <child link="tool0"/>
+    <origin rpy="0.08726646259971647 0 -3.141592653589793" xyz="0.0 -0.016124 -0.18430"/>
+  </joint>
   <!-- 'flange' frame: default pose reference frame -->
   <link name="flange" />
@@ -9,3 +21,11 @@
       prefix="$(arg prefix)"
       connected_to="$(arg prefix)flange"/>
+  <!-- Moveit Studio requires a link name called manual_grasp_link to
+       perform quick tasks such as inspect surface -->
+  <link name="manual_grasp_link" />
+  <joint name="$(arg prefix)manual_grasp_joint" type="fixed">
+    <origin xyz="0 0 0" rpy="0 0 0" />
+    <parent link="$(arg prefix)grasp_link" />
+    <child link="$(arg prefix)manual_grasp_link" />
+  </joint>
 </robot>
