Commit message: za6_tools:  Rotate hand-e gripper & move grasp link

File: za6_tools/urdf/robotiq_hand_e.urdf.xacro (robot description, xacro)
@@ -18,5 +18,5 @@
     <child link="tool0"/>
     <axis xyz="0 1 0"/>
-    <origin rpy="0 0 0" xyz="0 0 0"/>
+    <origin xyz="0 0 -0.135" rpy="0 0 ${pi/2.0}"/>
   </joint>
   <xacro:robotiq_hand_e_macro

File: za6_tools/urdf/robotiq_hand_e_macro.xacro (robot description, xacro)
@@ -14,5 +14,5 @@
           <mesh filename="package://za6_tools/meshes/robotiq_hand-e_gripper.stl"/>
         </geometry>
-        <origin rpy="0.0 0.0 0.0" xyz="0 0 0"/>
+        <origin xyz="0 0 0" rpy="0.0 0.0 0.0"/>
         <material name="${prefix}Black">
         </material>
@@ -22,5 +22,5 @@
           <mesh filename="package://za6_tools/meshes/robotiq_hand-e_gripper_collision.stl"/>
         </geometry>
-        <origin rpy="0.0 0.0 0.0" xyz="0 0 0"/>
+        <origin xyz="0 0 0" rpy="0.0 0.0 0.0"/>
       </collision>
       <inertial>
@@ -64,5 +64,5 @@
       <child link="${prefix}hand_e_body"/>
       <axis xyz="0 0 1"/>
-      <origin rpy="0 0 ${-pi/2.0}" xyz="0 0 0"/>
+      <origin xyz="0 0 0" rpy="0 0 ${-pi/2.0}"/>
     </joint>
     <joint name="${prefix}hand_e_body-hand_e_finger_left" type="fixed">
@@ -83,5 +83,5 @@
       <parent link="${prefix}hand_e_body" />
       <child link="grasp_link" />
-      <origin xyz="0.0 0.0 0.0" rpy="0.0 0.0 0.0" />
+      <origin xyz="0.0 0.0 0.135" rpy="0.0 0.0 0.0" />
     </joint>
   </xacro:macro>
