Commit message: za6_tools:  Unify top-level gripper urdf

File: za6_tools/urdf/gripper.urdf.xacro (robot description, xacro)
@@ -1,14 +1,14 @@
 <?xml version="1.0" ?>
-<robot name="za6_none" xmlns:xacro="http://www.ros.org/wiki/xacro">
-  <!-- URDF for *no* gripper:  no geometry; tool0 is at flange -->
+<robot xmlns:xacro="http://www.ros.org/wiki/xacro">
   <xacro:arg name="prefix" default=""/>
+  <xacro:arg name="gripper" default="pivot_gripper"/>
   <xacro:arg name="build" default="false"/>
   <xacro:if value="$(arg build)">
-    <xacro:include filename="$(cwd)/urdf/none_macro.xacro"/>
+    <xacro:property name="path_prefix" value="$(cwd)/urdf"/>
   </xacro:if>
   <xacro:unless value="$(arg build)">
-    <xacro:include
-        filename="$(find za6_tools)/urdf/none_macro.xacro"/>
+    <xacro:property name="path_prefix" value="$(find za6_tools)/urdf"/>
   </xacro:unless>
+  <xacro:include filename="${path_prefix}/$(arg gripper)_macro.xacro"/>
   <!-- Moveit Studio requires a link name called manual_grasp_link to
        perform quick tasks such as inspect surface -->
@@ -19,7 +19,9 @@
     <child link="tool0"/>
     <axis xyz="0 1 0"/>
-    <origin rpy="0 0 0" xyz="0.0 -0.016124 -0.18430"/>
+    <origin rpy="0 0 0" xyz="0 0 0"/>
   </joint>
-  <xacro:none_macro
+  <xacro:attribute name="name" value="za6_$(arg gripper)"/>
+  <xacro:element
+      xacro:name="xacro:$(arg gripper)_macro"
       prefix="$(arg prefix)"
       connected_to="$(arg prefix)tool0"/>

Commit message: za6_tools:  Add tests
Add tests similar to the `za6_description` package for testing URDFs
and launch files.

Fix a couple of problems in tests.

Update rviz config files.

Add `display_gripper.launch` notes to `README`.

File: za6_tools/urdf/gripper.urdf.xacro (robot description, xacro)
@@ -13,5 +13,5 @@
   <!-- Moveit Studio requires a link name called manual_grasp_link to
        perform quick tasks such as inspect surface -->
-  <link name="manual_grasp_link" />
+  <link name="manual_grasp_link"/>
   <link name="tool0"/>
   <joint name="tool0_joint" type="fixed">

File: za6_tools/urdf/none_macro.xacro (robot description, xacro)
@@ -9,5 +9,4 @@
       <parent link="${connected_to}"/>
       <child link="${prefix}grasp_link"/>
-      <axis xyz="0 0 0"/>
       <origin rpy="0.0 0.0 0.0" xyz="0 0 0"/>
     </joint>

File: za6_tools/urdf/pcnc1100/pcnc1100.urdf.xacro (robot description, xacro)
@@ -1,4 +1,5 @@
 <?xml version="1.0" ?>
 <robot name="pcnc1100" xmlns:xacro="http://www.ros.org/wiki/xacro">
+  <xacro:arg name="prefix" default=""/>
   <xacro:include
       filename="$(find za6_tools)/urdf/pcnc1100/pcnc1100_macro.xacro"/>
