Commit message: za6_tools:  Fix gripper URDF xacros for MoveIt Studio
Static URDF used as Studio `web_ui_gripper` was broken.  The iMarker
appeared at the robot base and couldn't be used to plan moves.

The meaningful change here is removing the joint that connected the
`grasp_link` link, which doesn't exist.

The versabuilt_multigrip is broken.  The scale looks off, it seems to
be missing `za6_multigrip_adapter` geometry incl. meshes, and
orientation is wrong.

File: za6_tools/config/robotiq_hand_e.srdf.xacro (robot description, xacro)
@@ -2,12 +2,12 @@
 <!--
 SRDF for the Robotiq Hand-E gripper
-To be used with the za6_tools package urdf/robotiq_hand_e_gripper.urdf.xacro
+To be used with the za6_tools package urdf/robotiq_hand_e.urdf.xacro
 -->
-<robot name="robotiq_hand_e_gripper" xmlns:xacro="http://www.ros.org/wiki/xacro">
+<robot name="robotiq_hand_e" xmlns:xacro="http://www.ros.org/wiki/xacro">
   <xacro:macro
-      name="robotiq_hand_e_gripper_macro"
+      name="robotiq_hand_e_macro"
       params="prefix robot_links:=${[]}">
     <!-- Gripper kinematic chain -->
-    <group name="${prefix}robotiq_hand_e_gripper">
+    <group name="${prefix}robotiq_hand_e">
       <link name="${prefix}hand_e_body"/>
       <link name="${prefix}hand_e_finger_left"/>
@@ -37,13 +37,13 @@
         <xacro:property name="robot_link" value="${robot_links.pop(0)}"/>
         <disable_collisions
-            link1="${prefix}flange-hand_e_body"
+            link1="${prefix}hand_e_body"
             link2="${robot_link}"
             reason="Never"/>
         <disable_collisions
-            link1="${prefix}hand_e_body-hand_e_finger_left"
+            link1="${prefix}hand_e_finger_left"
             link2="${robot_link}"
             reason="Never"/>
         <disable_collisions
-            link1="${prefix}hand_e_body-hand_e_finger_right"
+            link1="${prefix}hand_e_finger_right"
             link2="${robot_link}"
             reason="Never"/>

File: za6_tools/config/versabuilt_multigrip.srdf.xacro (robot description, xacro)
@@ -21,5 +21,5 @@
     <!-- Gripper internal collisions -->
     <disable_collisions
-        link1="${prefix}flange-multigrip_adapter"
+        link1="${prefix}multigrip_base_and_fixed_jaw"
         link2="${prefix}multigrip_moving_jaw"
         reason="Adjacent"/>

File: za6_tools/urdf/none.urdf.xacro (robot description, xacro)
@@ -8,24 +8,19 @@
   </xacro:if>
   <xacro:unless value="$(arg build)">
-    <xacro:include filename="$(find za6_tools)/urdf/none_macro.xacro"/>
+    <xacro:include
+        filename="$(find za6_tools)/urdf/none_macro.xacro"/>
   </xacro:unless>
-  <link name="tool0"/>
-  <joint name="flange-tool0" type="fixed">
-    <parent link="manual_grasp_link"/>
-    <child link="tool0"/>
-    <origin rpy="0 0 0" xyz="0.0 0.0 0.0"/>
-  </joint>
-  <!-- 'flange' frame: default pose reference frame -->
-  <link name="flange" />
-  <xacro:none_macro
-      prefix="$(arg prefix)"
-      connected_to="$(arg prefix)flange"/>
   <!-- Moveit Studio requires a link name called manual_grasp_link to
        perform quick tasks such as inspect surface -->
   <link name="manual_grasp_link" />
-  <joint name="grasp-manual_grasp" type="fixed">
-    <parent link="grasp_link"/>
-    <child link="manual_grasp_link"/>
-    <origin rpy="0 0 0" xyz="0.0 0.0 0.0"/>
+  <link name="tool0"/>
+  <joint name="tool0_joint" type="fixed">
+    <parent link="manual_grasp_link"/>
+    <child link="tool0"/>
+    <axis xyz="0 1 0"/>
+    <origin rpy="0 0 0" xyz="0.0 -0.016124 -0.18430"/>
   </joint>
+  <xacro:none_macro
+      prefix="$(arg prefix)"
+      connected_to="$(arg prefix)tool0"/>
 </robot>

File: za6_tools/urdf/none_macro.xacro (robot description, xacro)
@@ -3,5 +3,5 @@
   <xacro:macro name="none_macro" params="prefix connected_to">
     <!-- URDF for *no* gripper: define grasp_link with no geometry &
-         connect it -->
+         connect it at flange -->
     <link name="grasp_link"/>
     <!-- joint list -->

File: za6_tools/urdf/pivot_gripper.urdf.xacro (robot description, xacro)
@@ -7,24 +7,19 @@
   </xacro:if>
   <xacro:unless value="$(arg build)">
-    <xacro:include filename="$(cwd)/urdf/pivot_gripper_macro.xacro"/>
+    <xacro:include
+        filename="$(find za6_tools)/urdf/pivot_gripper_macro.xacro"/>
   </xacro:unless>
-  <link name="tool0"/>
-  <joint name="flange-tool0" type="fixed">
-    <parent link="manual_grasp_link"/>
-    <child link="tool0"/>
-    <origin rpy="0.08726646259971647 0 -3.141592653589793" xyz="0.0 -0.016124 -0.18430"/>
-  </joint>
-  <!-- 'flange' frame: default pose reference frame -->
-  <link name="flange" />
-  <xacro:pivot_gripper_macro
-      prefix="$(arg prefix)"
-      connected_to="$(arg prefix)flange"/>
   <!-- Moveit Studio requires a link name called manual_grasp_link to
        perform quick tasks such as inspect surface -->
   <link name="manual_grasp_link" />
-  <joint name="$(arg prefix)manual_grasp_joint" type="fixed">
-    <origin xyz="0 0 0" rpy="0 0 0" />
-    <parent link="$(arg prefix)grasp_link" />
-    <child link="$(arg prefix)manual_grasp_link" />
+  <link name="tool0"/>
+  <joint name="tool0_joint" type="fixed">
+    <parent link="manual_grasp_link"/>
+    <child link="tool0"/>
+    <axis xyz="0 1 0"/>
+    <origin rpy="0 0 0" xyz="0 0 0"/>
   </joint>
+  <xacro:pivot_gripper_macro
+      prefix="$(arg prefix)"
+      connected_to="$(arg prefix)tool0"/>
 </robot>

File: za6_tools/urdf/robotiq_hand_e.urdf.xacro (robot description, xacro)
@@ -7,24 +7,19 @@
   </xacro:if>
   <xacro:unless value="$(arg build)">
-    <xacro:include filename="$(find za6_tools)/urdf/robotiq_hand_e_macro.xacro"/>
+    <xacro:include
+        filename="$(find za6_tools)/urdf/robotiq_hand_e_macro.xacro"/>
   </xacro:unless>
-  <link name="tool0"/>
-  <joint name="flange-tool0" type="fixed">
-    <parent link="manual_grasp_link"/>
-    <child link="tool0"/>
-    <origin rpy="0.08726646259971647 0 -3.141592653589793" xyz="0.0 -0.016124 -0.18430"/>
-  </joint>
-  <!-- 'flange' frame: default pose reference frame -->
-  <link name="flange" />
-  <xacro:robotiq_hand_e_macro
-      prefix="$(arg prefix)"
-      connected_to="$(arg prefix)flange"/>
   <!-- Moveit Studio requires a link name called manual_grasp_link to
        perform quick tasks such as inspect surface -->
   <link name="manual_grasp_link" />
-  <joint name="$(arg prefix)manual_grasp_joint" type="fixed">
-    <origin xyz="0 0 0" rpy="0 0 0" />
-    <parent link="$(arg prefix)grasp_link" />
-    <child link="$(arg prefix)manual_grasp_link" />
+  <link name="tool0"/>
+  <joint name="tool0_joint" type="fixed">
+    <parent link="manual_grasp_link"/>
+    <child link="tool0"/>
+    <axis xyz="0 1 0"/>
+    <origin rpy="0 0 0" xyz="0 0 0"/>
   </joint>
+  <xacro:robotiq_hand_e_macro
+      prefix="$(arg prefix)"
+      connected_to="$(arg prefix)tool0"/>
 </robot>

File: za6_tools/urdf/versabuilt_multigrip.urdf.xacro (robot description, xacro)
@@ -10,22 +10,16 @@
         filename="$(find za6_tools)/urdf/versabuilt_multigrip_macro.xacro"/>
   </xacro:unless>
-  <link name="tool0"/>
-  <joint name="flange-tool0" type="fixed">
-    <parent link="manual_grasp_link"/>
-    <child link="tool0"/>
-    <origin rpy="0.08726646259971647 0 -3.141592653589793" xyz="0.0 -0.016124 -0.18430"/>
-  </joint>
-  <!-- 'flange' frame: default pose reference frame -->
-  <link name="flange" />
-  <xacro:versabuilt_multigrip_macro
-      prefix="$(arg prefix)"
-      connected_to="$(arg prefix)flange"/>
   <!-- Moveit Studio requires a link name called manual_grasp_link to
        perform quick tasks such as inspect surface -->
   <link name="manual_grasp_link" />
-  <joint name="$(arg prefix)manual_grasp_joint" type="fixed">
-    <origin xyz="0 0 0" rpy="0 0 0" />
-    <parent link="$(arg prefix)grasp_link" />
-    <child link="$(arg prefix)manual_grasp_link" />
+  <link name="tool0"/>
+  <joint name="tool0_joint" type="fixed">
+    <parent link="manual_grasp_link"/>
+    <child link="tool0"/>
+    <axis xyz="0 1 0"/>
+    <origin rpy="${pi/36} 0 -${pi}" xyz="0.0 -0.016124 -0.18430"/>
   </joint>
+  <xacro:versabuilt_multigrip_macro
+      prefix="$(arg prefix)"
+      connected_to="$(arg prefix)tool0"/>
 </robot>

File: za6_tools/urdf/versabuilt_multigrip_macro.xacro (robot description, xacro)
@@ -6,6 +6,5 @@
     </material>
     <!-- link list -->
-    <link name="${prefix}za6_multigrip_adapter">
-    </link>
+    <link name="${prefix}za6_multigrip_adapter"/>
     <link name="${prefix}multigrip_base_and_fixed_jaw">
       <visual>
