Commit message: za6_moveit_config:  Fix SRDF robot mount collisions
The robot base (i.e. whatever the robot is mounted on) may have a
collision model that intersects the robot's base link (i.e. the link
under `link_1`).

The `MoveItConfigsBuilder` class (used in
e.g. `launch/static_virtual_joint_tfs.launch.py`) and MoveIt Studio
configs all need static SRDFs at run time.  To accomplish this for the
former, render a basic SRDF into `config/za6.srdf`, and for the
latter, provide a CMake function for generating SRDFs for the ZA6 and
each gripper in the `za6_tools` package, plus a configurable robot
base link.

File: za6_moveit_config/config/za6.srdf.xacro (robot description, xacro)
@@ -9,4 +9,5 @@
   <xacro:arg name="prefix" default=""/>
   <xacro:arg name="gripper" default="none"/>
+  <xacro:arg name="mount_link" default=""/>
   <!-- Main manipulator move group -->
   <group name="manipulator">
@@ -38,4 +39,10 @@
   <disable_collisions link1="link_4" link2="link_6" reason="User"/>
   <disable_collisions link1="link_5" link2="link_6" reason="Adjacent"/>
+  <!-- Robot mount -->
+  <xacro:property name="mount_link" value="$(arg mount_link)"/>
+  <xacro:if value="${mount_link != ''}">
+    <!-- Robot base may intersect with mount collision model -->
+    <disable_collisions link1="base_link" link2="${mount_link}" reason="Adjacent"/>
+  </xacro:if>
   <!-- Gripper macros -->
   <xacro:property name="gripper" value="$(arg gripper)"/>
