Commit message: moveit_studio_za6_tending_config:  Update URDF and SRDF
Replace UR5e with ZA6

File: moveit_studio_za6_tending_config/description/za6_machine_tending.xacro (robot description, xacro)
@@ -1,7 +1,40 @@
 <?xml version="1.0"?>
-<robot xmlns:xacro="http://wiki.ros.org/xacro" name="$(arg name)">
-  <!-- parameters -->
-  <xacro:arg name="use_fake_hardware" default="false" />
-  <xacro:arg name="external_camera" default="false" />
+<robot name="za6" xmlns:xacro="http://www.ros.org/wiki/xacro">
+  <!-- ZA6-specific parameters -->
+  <xacro:arg name="prefix" default=""/>
+  <xacro:arg name="fixed_tool" default="True"/>
+  <xacro:arg name="include_ros2_control" default="False"/>
+  <xacro:arg name="ros2_control_name" default="hal_hw_interface"/>
+  <xacro:arg name="ros2_control_plugin"
+             default="hal_system_interface/HalSystemInterface"/>
+  <!-- Used by ros2_control fake hardware -->
+  <xacro:arg name="initial_positions_file"
+             default="$(find za6_description)/config/initial_positions.yaml"/>
+  <xacro:arg name="limit_joint_1_lower" default="-2.96"/>
+  <xacro:arg name="limit_joint_1_upper" default="2.96"/>
+  <xacro:arg name="limit_joint_1_velocity" default="2.0"/>
+  <xacro:arg name="limit_joint_1_effort" default="1000.0"/>
+  <xacro:arg name="limit_joint_2_lower" default="-1.74"/>
+  <xacro:arg name="limit_joint_2_upper" default="2.35"/>
+  <xacro:arg name="limit_joint_2_velocity" default="3.1"/>
+  <xacro:arg name="limit_joint_2_effort" default="1000.0"/>
+  <xacro:arg name="limit_joint_3_lower" default="-3.7"/>
+  <xacro:arg name="limit_joint_3_upper" default="1.15"/>
+  <xacro:arg name="limit_joint_3_velocity" default="3.9"/>
+  <xacro:arg name="limit_joint_3_effort" default="1000.0"/>
+  <xacro:arg name="limit_joint_4_lower" default="-2.6"/>
+  <xacro:arg name="limit_joint_4_upper" default="2.6"/>
+  <xacro:arg name="limit_joint_4_velocity" default="3.0"/>
+  <xacro:arg name="limit_joint_4_effort" default="1000.0"/>
+  <xacro:arg name="limit_joint_5_lower" default="-2.49"/>
+  <xacro:arg name="limit_joint_5_upper" default="2.49"/>
+  <xacro:arg name="limit_joint_5_velocity" default="3.8"/>
+  <xacro:arg name="limit_joint_5_effort" default="1000.0"/>
+  <xacro:arg name="limit_joint_6_lower" default="-6.283"/>
+  <xacro:arg name="limit_joint_6_upper" default="6.283"/>
+  <xacro:arg name="limit_joint_6_velocity" default="6.2"/>
+  <xacro:arg name="limit_joint_6_effort" default="1000.0"/>
+  <!-- Other parameters -->
+  <!-- <xacro:arg name="use_fake_hardware" default="false" /> -->
   <xacro:arg name="has_tool_changer" default="true" />
   <xacro:arg name="use_pinch_links" default="true" />
@@ -27,26 +60,11 @@
   <xacro:include filename="$(find picknik_accessories)/descriptions/sensors/realsense_d415.urdf.xacro" />
   <xacro:include filename="$(find picknik_ur_base_config)/description/pinch_links.xacro" />
+  <xacro:include
+      filename="$(find za6_description)/urdf/za6_macro.xacro"/>
   <!-- Initial positions for simulations (Mock Hardware and Gazebo) -->
-  <xacro:arg name="initial_positions_file" default="$(find za6_machine_tending_config)/config/initial_positions.yaml"/>
-  <xacro:property name="initial_positions_file" default="$(arg initial_positions_file)"/>
+  <xacro:property
+      name="initial_positions_file"
+      default="$(arg initial_positions_file)"/>
   <link name="world" />
-  <!-- arm -->
-  <xacro:ur_robot
-    name="$(arg name)"
-    tf_prefix=""
-    parent="world"
-    joint_limits_parameters_file="$(arg joint_limits_parameters_file)"
-    kinematics_parameters_file="$(arg kinematics_parameters_file)"
-    physical_parameters_file="$(arg physical_parameters_file)"
-    visual_parameters_file="$(arg visual_parameters_file)"
-    use_fake_hardware="$(arg use_fake_hardware)"
-    initial_positions="${xacro.load_yaml(initial_positions_file)}"
-    headless_mode="$(arg headless_mode)"
-    robot_ip="$(arg robot_ip)"
-    script_filename="$(find ur_robot_driver)/resources/ros_control.urscript"
-    output_recipe_filename="$(find ur_robot_driver)/resources/rtde_output_recipe.txt"
-    input_recipe_filename="$(find ur_robot_driver)/resources/rtde_input_recipe.txt">
-    <origin xyz="0 0 0" rpy="0 0 ${pi/2}" />
-  </xacro:ur_robot>
   <xacro:if value="$(arg has_tool_changer)">
     <!-- tool changer-->
@@ -74,6 +92,41 @@
     <child link="grasp_link" />
     <origin xyz="0.0 0.0 0.134" rpy="0.0 0.0 ${pi}" />
-  </joint>
-  <!-- Moveit Studio requires a link name called manual_grasp_link to perform quick tasks such as inspect surface -->
+  <joint name="world-$(arg prefix)base_link" type="fixed">
+    <origin xyz="0 0 0" rpy="0 0 -${pi/2}"/>
+    <axis xyz="0 0 1"/>
+    <parent link="world"/>
+    <child link="$(arg prefix)base_link"/>
+  </joint>
+  <!-- arm -->
+  <xacro:za6
+      prefix="$(arg prefix)"
+      tool0_trans="0 0 0"
+      tool0_rot="0 0 0"
+      tool0_fixed="$(arg fixed_tool)"
+      limit_joint_1_lower="$(arg limit_joint_1_lower)"
+      limit_joint_1_upper="$(arg limit_joint_1_upper)"
+      limit_joint_1_velocity="$(arg limit_joint_1_velocity)"
+      limit_joint_1_effort="$(arg limit_joint_1_effort)"
+      limit_joint_2_lower="$(arg limit_joint_2_lower)"
+      limit_joint_2_upper="$(arg limit_joint_2_upper)"
+      limit_joint_2_velocity="$(arg limit_joint_2_velocity)"
+      limit_joint_2_effort="$(arg limit_joint_2_effort)"
+      limit_joint_3_lower="$(arg limit_joint_3_lower)"
+      limit_joint_3_upper="$(arg limit_joint_3_upper)"
+      limit_joint_3_velocity="$(arg limit_joint_3_velocity)"
+      limit_joint_3_effort="$(arg limit_joint_3_effort)"
+      limit_joint_4_lower="$(arg limit_joint_4_lower)"
+      limit_joint_4_upper="$(arg limit_joint_4_upper)"
+      limit_joint_4_velocity="$(arg limit_joint_4_velocity)"
+      limit_joint_4_effort="$(arg limit_joint_4_effort)"
+      limit_joint_5_lower="$(arg limit_joint_5_lower)"
+      limit_joint_5_upper="$(arg limit_joint_5_upper)"
+      limit_joint_5_velocity="$(arg limit_joint_5_velocity)"
+      limit_joint_5_effort="$(arg limit_joint_5_effort)"
+      limit_joint_6_lower="$(arg limit_joint_6_lower)"
+      limit_joint_6_upper="$(arg limit_joint_6_upper)"
+      limit_joint_6_velocity="$(arg limit_joint_6_velocity)"
+      limit_joint_6_effort="$(arg limit_joint_6_effort)"
+      />
   <link name="manual_grasp_link" />
   <joint name="manual_grasp_joint" type="fixed">
@@ -81,4 +134,8 @@
     <child link="manual_grasp_link" />
     <origin xyz="0 0 0" rpy="${pi / 180.0 * 5} 0 0" />
+  <joint name="$(arg prefix)manual_grasp_link-tool0" type="fixed">
+    <origin xyz="0 0 0" rpy="0 0 0" />
+    <parent link="$(arg prefix)tool0" />
+    <child link="$(arg prefix)manual_grasp_link" />
   </joint>
   <!-- CNC machine -->
@@ -87,5 +144,7 @@
       <origin xyz="0 0 0" rpy="0 0 0" />
       <geometry>
-        <mesh filename="file://$(find za6_machine_tending_config)/meshes/cnc.dae" scale="1 1 1"/>
+        <mesh
+            filename="file://$(find moveit_studio_za6_tending_config)/meshes/cnc.dae"
+            scale="1 1 1"/>
       </geometry>
     </visual>
@@ -94,5 +153,7 @@
       <origin xyz="0 0 0" rpy="0 0 0"/>
       <geometry>
-        <mesh filename="file://$(find za6_machine_tending_config)/meshes/cnc-collision.dae" scale="1 1 1"/>
+        <mesh
+            filename="file://$(find moveit_studio_za6_tending_config)/meshes/cnc-collision.dae"
+            scale="1 1 1"/>
       </geometry>
     </collision>
@@ -108,5 +169,7 @@
       <origin xyz="0 0 0" rpy="0 0 0" />
       <geometry>
-        <mesh filename="file://$(find za6_machine_tending_config)/meshes/base.dae" scale="1 1 1"/>
+        <mesh
+            filename="file://$(find moveit_studio_za6_tending_config)/meshes/base.dae"
+            scale="1 1 1"/>
       </geometry>
     </visual>
@@ -114,5 +177,7 @@
       <origin xyz="0 0 0" rpy="0 0 0"/>
       <geometry>
-        <mesh filename="file://$(find za6_machine_tending_config)/meshes/base.dae" scale="1 1 1"/>
+        <mesh
+            filename="file://$(find moveit_studio_za6_tending_config)/meshes/base.dae"
+            scale="1 1 1"/>
       </geometry>
     </collision>
@@ -128,11 +193,15 @@
       <origin xyz="0 0 0" rpy="0 0 0" />
       <geometry>
-        <mesh filename="file://$(find za6_machine_tending_config)/meshes/table.dae" scale="1 1 1"/>
-      </geometry>
-    </visual>
-    <collision>
-      <origin xyz="0 0 0" rpy="0 0 0" />
-      <geometry>
-        <mesh filename="file://$(find za6_machine_tending_config)/meshes/table-collision.dae" scale="1 1 1"/>
+        <mesh
+            filename="file://$(find moveit_studio_za6_tending_config)/meshes/table.dae"
+            scale="1 1 1"/>
+      </geometry>
+    </visual>
+    <collision>
+      <origin xyz="0 0 0" rpy="0 0 0" />
+      <geometry>
+        <mesh
+            filename="file://$(find moveit_studio_za6_tending_config)/meshes/table-collision.dae"
+            scale="1 1 1"/>
       </geometry>
     </collision>
@@ -147,11 +216,15 @@
       <origin xyz="0 0 0" rpy="0 0 0" />
       <geometry>
-        <mesh filename="file://$(find za6_machine_tending_config)/meshes/table.dae" scale="1 1 1"/>
-      </geometry>
-    </visual>
-    <collision>
-      <origin xyz="0 0 0" rpy="0 0 0" />
-      <geometry>
-        <mesh filename="file://$(find za6_machine_tending_config)/meshes/table-collision.dae" scale="1 1 1"/>
+        <mesh
+            filename="file://$(find moveit_studio_za6_tending_config)/meshes/table.dae"
+            scale="1 1 1"/>
+      </geometry>
+    </visual>
+    <collision>
+      <origin xyz="0 0 0" rpy="0 0 0" />
+      <geometry>
+        <mesh
+            filename="file://$(find moveit_studio_za6_tending_config)/meshes/table-collision.dae"
+            scale="1 1 1"/>
       </geometry>
     </collision>
@@ -167,5 +240,7 @@
       <origin xyz="0 0 0" rpy="0 0 0" />
       <geometry>
-        <mesh filename="file://$(find za6_machine_tending_config)/meshes/cylinder-item.dae" scale="1 1 1"/>
+        <mesh
+            filename="file://$(find moveit_studio_za6_tending_config)/meshes/cylinder-item.dae"
+            scale="1 1 1"/>
       </geometry>
     </visual>
@@ -181,5 +256,7 @@
       <origin xyz="0 0 0" rpy="0 0 0" />
       <geometry>
-        <mesh filename="file://$(find za6_machine_tending_config)/meshes/cylinder-item.dae" scale="1 1 1"/>
+        <mesh
+            filename="file://$(find moveit_studio_za6_tending_config)/meshes/cylinder-item.dae"
+            scale="1 1 1"/>
       </geometry>
     </visual>

Commit message: Import za6_tools package
Pulled in from ROS (1) repo commit 7374754c5

File: moveit_studio_za6_tending_config/description/za6_machine_tending.xacro (robot description, xacro)
@@ -37,28 +37,6 @@
   <xacro:arg name="limit_joint_6_effort" default="1000.0"/>
   <!-- Other parameters -->
-  <!-- <xacro:arg name="use_fake_hardware" default="false" /> -->
-  <xacro:arg name="has_tool_changer" default="true" />
-  <xacro:arg name="use_pinch_links" default="true" />
-  <xacro:arg name="name" default="" />
-  <xacro:arg name="joint_limits_parameters_file" default="" />
-  <xacro:arg name="kinematics_parameters_file" default="" />
-  <xacro:arg name="physical_parameters_file" default="" />
-  <xacro:arg name="visual_parameters_file" default="" />
-  <xacro:arg name="headless_mode" default="false" />
-  <xacro:arg name="robot_ip" default="0.0.0.0" />
-  <xacro:if value="$(arg has_tool_changer)">
-    <xacro:property name="camera_adapter_parent" value="tool_changer_tool0" />
-  </xacro:if>
-  <xacro:unless value="$(arg has_tool_changer)">
-    <xacro:property name="camera_adapter_parent" value="tool0" />
-  </xacro:unless>
+  <xacro:property name="camera_adapter_parent" value="tool0" />
   <!-- Import macros for main hardware components -->
-  <xacro:include filename="$(find ur_description)/urdf/ur_macro.xacro" />
-  <xacro:include filename="$(find robotiq_description)/urdf/ur_to_robotiq_adapter.urdf.xacro" />
-  <xacro:include filename="$(find robotiq_description)/urdf/robotiq_2f_85_macro.urdf.xacro" />
-  <xacro:include filename="$(find picknik_accessories)/descriptions/brackets/mtc_ur_tool_changer/mtc_ur_tool_changer.urdf.xacro" />
-  <xacro:include filename="$(find picknik_accessories)/descriptions/brackets/ur_realsense_camera_adapter/picknik_ur_camera_adapter.urdf.xacro" />
-  <xacro:include filename="$(find picknik_accessories)/descriptions/sensors/realsense_d415.urdf.xacro" />
-  <xacro:include filename="$(find picknik_ur_base_config)/description/pinch_links.xacro" />
   <xacro:include
       filename="$(find za6_description)/urdf/za6_macro.xacro"/>
@@ -68,29 +46,4 @@
       default="$(arg initial_positions_file)"/>
   <link name="world" />
-  <xacro:if value="$(arg has_tool_changer)">
-    <!-- tool changer-->
-    <xacro:mtc_ur_tool_changer prefix="" connected_to="tool0" rotation="0" />
-  </xacro:if>
-  <!-- pinch geometry for moveit motion planning. see https://github.com/UniversalRobots/Universal_Robots_ROS2_Driver/issues/611 -->
-  <xacro:if value="$(arg use_pinch_links)">
-    <xacro:forearm_pinch_link />
-    <xacro:wrist_3_pinch_link />
-  </xacro:if>
-  <!-- wrist camera adapter and camera-->
-  <xacro:ur_realsense_camera_adapter prefix="" connected_to="${camera_adapter_parent}" rotation="0" />
-  <xacro:realsense_d415 parent="d415_mount_link" name="wrist_mounted_camera">
-    <origin xyz="0 0 0" rpy="0 0 0" />
-  </xacro:realsense_d415>
-  <!-- Gripper and UR adapter-->
-  <xacro:ur_to_robotiq prefix="" connected_to="realsense_camera_adapter_tool0" rotation="0" />
-  <xacro:robotiq_gripper name="RobotiqGripperHardwareInterface" prefix=""
-    parent="gripper_mount_link" use_fake_hardware="$(arg use_fake_hardware)" com_port="/dev/ttyUSB0">
-    <origin xyz="0 0 0" rpy="0 0 0" />
-  </xacro:robotiq_gripper>
-  <link name="grasp_link" />
-  <joint name="grasp_link_joint" type="fixed">
-    <parent link="gripper_mount_link" />
-    <child link="grasp_link" />
-    <origin xyz="0.0 0.0 0.134" rpy="0.0 0.0 ${pi}" />
   <joint name="world-$(arg prefix)base_link" type="fixed">
     <origin xyz="0 0 0" rpy="0 0 -${pi/2}"/>
@@ -130,13 +83,54 @@
       limit_joint_6_effort="$(arg limit_joint_6_effort)"
       />
+  <!-- ros2_control -->
+  <xacro:if value="$(arg include_ros2_control)">
+    <xacro:include filename="$(find za6_description)/urdf/za6.ros2_control.xacro"/>
+    <xacro:za6_ros2_control
+        name="$(arg ros2_control_name)"
+        prefix="$(arg prefix)"
+        initial_positions_file="$(arg initial_positions_file)"
+        use_mock_hardware="$(arg use_mock_hardware)"
+        ros2_control_plugin="$(arg ros2_control_plugin)"
+        limit_joint_1_lower="$(arg limit_joint_1_lower)"
+        limit_joint_1_upper="$(arg limit_joint_1_upper)"
+        limit_joint_1_velocity="$(arg limit_joint_1_velocity)"
+        limit_joint_2_lower="$(arg limit_joint_2_lower)"
+        limit_joint_2_upper="$(arg limit_joint_2_upper)"
+        limit_joint_2_velocity="$(arg limit_joint_2_velocity)"
+        limit_joint_3_lower="$(arg limit_joint_3_lower)"
+        limit_joint_3_upper="$(arg limit_joint_3_upper)"
+        limit_joint_3_velocity="$(arg limit_joint_3_velocity)"
+        limit_joint_4_lower="$(arg limit_joint_4_lower)"
+        limit_joint_4_upper="$(arg limit_joint_4_upper)"
+        limit_joint_4_velocity="$(arg limit_joint_4_velocity)"
+        limit_joint_5_lower="$(arg limit_joint_5_lower)"
+        limit_joint_5_upper="$(arg limit_joint_5_upper)"
+        limit_joint_5_velocity="$(arg limit_joint_5_velocity)"
+        limit_joint_6_lower="$(arg limit_joint_6_lower)"
+        limit_joint_6_upper="$(arg limit_joint_6_upper)"
+        limit_joint_6_velocity="$(arg limit_joint_6_velocity)"
+        />
+  </xacro:if>
+  <!-- Gripper -->
+  <xacro:include
+      filename="$(find za6_tools)/urdf/pivot_gripper_macro.xacro" />
+  <!-- Attach Pivot gripper to ZA6 "flange" link -->
+  <xacro:pivot_gripper_macro
+      prefix="$(arg prefix)"
+      connected_to="$(arg prefix)flange"/>
+  <!-- Attach grasp_link to gripper base for now -->
+  <link name="grasp_link" />
+  <joint name="grasp_link_joint" type="fixed">
+    <parent link="$(arg prefix)pivot_gripper_base" />
+    <child link="grasp_link" />
+    <origin xyz="0.0 0.0 0.0" rpy="0.0 0.0 0.0" />
+  </joint>
+  <!-- Moveit Studio requires a link name called manual_grasp_link to
+       perform quick tasks such as inspect surface -->
   <link name="manual_grasp_link" />
   <joint name="manual_grasp_joint" type="fixed">
     <parent link="grasp_link" />
     <child link="manual_grasp_link" />
-    <origin xyz="0 0 0" rpy="${pi / 180.0 * 5} 0 0" />
-  <joint name="$(arg prefix)manual_grasp_link-tool0" type="fixed">
     <origin xyz="0 0 0" rpy="0 0 0" />
-    <parent link="$(arg prefix)tool0" />
-    <child link="$(arg prefix)manual_grasp_link" />
   </joint>
   <!-- CNC machine -->

File: za6_description/urdf/za6.xacro (robot description, xacro)
@@ -2,5 +2,5 @@
 <robot name="za6" xmlns:xacro="http://www.ros.org/wiki/xacro">
   <xacro:arg name="prefix" default=""/>
-  <xacro:arg name="fixed_tool" default="True"/>
+  <xacro:arg name="fixed_tool" default="true"/>
   <xacro:arg name="include_ros2_control" default="false"/>
   <xacro:arg name="ros2_control_name" default="hal_hw_interface"/>

File: za6_description/urdf/za6_macro.xacro (robot description, xacro)
@@ -2,5 +2,6 @@
 <robot xmlns:xacro="http://www.ros.org/wiki/xacro">
   <xacro:macro name="za6" params="
-    prefix tool0_trans tool0_rot tool0_fixed
+    prefix tool0_trans tool0_rot
+    tool0_fixed:=True
     limit_joint_1_lower:=-2.96
     limit_joint_1_upper:=2.96

Commit message: Make base & tending .xacro files directly diffable
Helps troubleshooting.  Would be nice if the rest of the
diffs (gripper, PCNC, table, etc.) could be brought in with a short
`xacro` macro.

File: moveit_studio_za6_tending_config/description/za6_machine_tending.xacro (robot description, xacro)
@@ -1,8 +1,7 @@
 <?xml version="1.0"?>
 <robot name="za6" xmlns:xacro="http://www.ros.org/wiki/xacro">
-  <!-- ZA6-specific parameters -->
   <xacro:arg name="prefix" default=""/>
-  <xacro:arg name="fixed_tool" default="True"/>
-  <xacro:arg name="include_ros2_control" default="False"/>
+  <xacro:arg name="fixed_tool" default="true"/>
+  <xacro:arg name="include_ros2_control" default="false"/>
   <xacro:arg name="ros2_control_name" default="hal_hw_interface"/>
   <xacro:arg name="use_mock_hardware" default="false"/>
@@ -36,21 +35,13 @@
   <xacro:arg name="limit_joint_6_velocity" default="6.2"/>
   <xacro:arg name="limit_joint_6_effort" default="1000.0"/>
-  <!-- Other parameters -->
-  <xacro:property name="camera_adapter_parent" value="tool0" />
-  <!-- Import macros for main hardware components -->
-  <xacro:include
-      filename="$(find za6_description)/urdf/za6_macro.xacro"/>
-  <!-- Initial positions for simulations (Mock Hardware and Gazebo) -->
-  <xacro:property
-      name="initial_positions_file"
-      default="$(arg initial_positions_file)"/>
-  <link name="world" />
-  <joint name="world-$(arg prefix)base_link" type="fixed">
-    <origin xyz="0 0 0" rpy="0 0 -${pi/2}"/>
-    <axis xyz="0 0 1"/>
-    <parent link="world"/>
-    <child link="$(arg prefix)base_link"/>
-  </joint>
-  <!-- arm -->
+  <xacro:arg name="gripper" default=""/>
+  <xacro:property name="gripper" value="$(arg gripper)"/>
+  <xacro:unless value="${gripper == '' or gripper == 'none'}">
+    <!-- MoveIt Studio web preview gripper model -->
+    <xacro:attribute
+        name="web_ui_gripper"
+        value="$(find za6_tools)/urdf/${gripper}_macro.xacro"/>
+  </xacro:unless>
+  <xacro:include filename="$(find za6_description)/urdf/za6_macro.xacro"/>
   <xacro:za6
       prefix="$(arg prefix)"
@@ -58,4 +49,5 @@
       tool0_rot="0 0 0"
       tool0_fixed="$(arg fixed_tool)"
+      gripper="${gripper}"
       limit_joint_1_lower="$(arg limit_joint_1_lower)"
       limit_joint_1_upper="$(arg limit_joint_1_upper)"
@@ -112,26 +104,23 @@
         />
   </xacro:if>
-  <!-- Gripper -->
-  <xacro:include
-      filename="$(find za6_tools)/urdf/pivot_gripper_macro.xacro" />
-  <!-- Attach Pivot gripper to ZA6 "flange" link -->
-  <xacro:pivot_gripper_macro
-      prefix="$(arg prefix)"
-      connected_to="$(arg prefix)flange"/>
-  <!-- Attach grasp_link to gripper base for now -->
-  <link name="grasp_link" />
-  <joint name="grasp_link_joint" type="fixed">
-    <parent link="$(arg prefix)pivot_gripper_base" />
-    <child link="grasp_link" />
-    <origin xyz="0.0 0.0 0.0" rpy="0.0 0.0 0.0" />
+  <!-- 'world' frame: default pose reference frame -->
+  <link name="world" />
+  <joint name="world-$(arg prefix)base_link" type="fixed">
+    <origin xyz="0 0 0" rpy="0 0 -${pi/2}"/>
+    <axis xyz="0 0 1"/>
+    <parent link="world"/>
+    <child link="$(arg prefix)base_link"/>
   </joint>
   <!-- Moveit Studio requires a link name called manual_grasp_link to
        perform quick tasks such as inspect surface -->
   <link name="manual_grasp_link" />
-  <joint name="manual_grasp_joint" type="fixed">
-    <parent link="grasp_link" />
-    <child link="manual_grasp_link" />
+  <joint name="$(arg prefix)manual_grasp_joint" type="fixed">
     <origin xyz="0 0 0" rpy="0 0 0" />
-  </joint>
+    <parent link="$(arg prefix)grasp_link" />
+    <child link="$(arg prefix)manual_grasp_link" />
+  </joint>
+  <xacro:attribute
+      name="web_ui_gripper"
+      value="file://$(find za6_tools)/urdf/$(arg gripper).urdf"/>
   <!-- CNC machine -->
   <link name="cnc_machine">

File: za6_description/urdf/za6.xacro (robot description, xacro)
@@ -1,3 +1,3 @@
-<?xml version="1.0" ?>
+<?xml version="1.0"?>
 <robot name="za6" xmlns:xacro="http://www.ros.org/wiki/xacro">
   <xacro:arg name="prefix" default=""/>
@@ -103,7 +103,8 @@
     <child link="$(arg prefix)base_link"/>
   </joint>
-  <!-- MoveIt Studio 'manual_grasp_link' for planning -->
+  <!-- Moveit Studio requires a link name called manual_grasp_link to
+       perform quick tasks such as inspect surface -->
   <link name="manual_grasp_link" />
-  <joint name="$(arg prefix)manual_grasp_link-tool0" type="fixed">
+  <joint name="$(arg prefix)manual_grasp_joint" type="fixed">
     <origin xyz="0 0 0" rpy="0 0 0" />
     <parent link="$(arg prefix)tool0" />
