Commit message: moveit_studio_za6_tending_config:  Fix SRDF
Collision btw robot mount base and robot broke MoveIt planning.

Fix it by pulling in SRDF generation macros from `za6_moveit_config`
pkg that disable collision checking for the robot mount.

Add other minor fixups to the URDF.

File: moveit_studio_za6_tending_config/description/za6_machine_tending.xacro (robot description, xacro)
@@ -35,12 +35,9 @@
   <xacro:arg name="limit_joint_6_velocity" default="6.2"/>
   <xacro:arg name="limit_joint_6_effort" default="1000.0"/>
-  <xacro:arg name="gripper" default=""/>
-  <xacro:property name="gripper" value="$(arg gripper)"/>
-  <xacro:unless value="${gripper == '' or gripper == 'none'}">
-    <!-- MoveIt Studio web preview gripper model -->
-    <xacro:attribute
-        name="web_ui_gripper"
-        value="$(find za6_tools)/urdf/${gripper}_macro.xacro"/>
-  </xacro:unless>
+  <xacro:arg name="gripper" default="none"/>
+  <!-- MoveIt Studio web preview gripper model -->
+  <xacro:attribute
+      name="web_ui_gripper"
+      value="package://za6_tools/urdf/$(arg gripper).urdf"/>
   <xacro:include filename="$(find za6_description)/urdf/za6_macro.xacro"/>
   <xacro:za6
@@ -49,5 +46,5 @@
       tool0_rot="0 0 0"
       tool0_fixed="$(arg fixed_tool)"
-      gripper="${gripper}"
+      gripper="$(arg gripper)"
       limit_joint_1_lower="$(arg limit_joint_1_lower)"
       limit_joint_1_upper="$(arg limit_joint_1_upper)"
@@ -120,7 +117,4 @@
     <child link="$(arg prefix)manual_grasp_link" />
   </joint>
-  <xacro:attribute
-      name="web_ui_gripper"
-      value="file://$(find za6_tools)/urdf/$(arg gripper).urdf"/>
   <!-- CNC machine -->
   <link name="cnc_machine">
